File: pi-filter-busboard.kicad_pcb (KiCad board)
At the start: 2 copper layers, 371 x 40 mm, 44 parts, among them J1 IDC_2x5, J10 IDC_2x5, J11 IDC_2x8, J12 IDC_2x8, J13 IDC_2x5, J14 IDC_2x5, J15 IDC_2x5, J16 IDC_2x5, J17 IDC_2x5, J18 IDC_2x5, J19 IDC_2x5, J2 IDC_2x5, J20 IDC_2x5, J21 IDC_2x5, J22 IDC_2x5, J23 Screw_Terminal_01x03, J3 IDC_2x5, J4 IDC_2x5, J5 IDC_2x5, J6 IDC_2x5, J7 IDC_2x5, J8 IDC_2x5, J9 IDC_2x5, U1 OKI-78SR-5_1.5-W36-C

Commit message: Update PCB layout
Parts:
- renumbered +12v1 to +12v, +5v1 to +5v, -12v1 to -12v
